File: hw/RC_module.brd (EAGLE design)
At the start: 40 x 40 mm, 32 parts, among them U1 STM32F103CX, U5 LD3985XX, X1 MICROMATCH-4

Commit message: layout completed
Parts:
- removed R3: 100k, rcl:R0603
- removed X1: MICROMATCH-4, tyco:MICROMATCH-4
- added RN1, RN2, RN3: (no value), dp_devices:RN8P-4R-CRA06S
- added U$10, U$11, U$12, U$13, U$14, U$2, U$3, U$5, U$6, U$7, U$8, U$9: PINHD-3, connectors:1X03
- added U$15: SCREWTERMINAL_3-3, connectors:SCREWTERMINAL-3.5MM-2
- C11: value 15pF -> 10n
- moved C11 6.76 mm to (27.1, 29.8), turned to 270 degrees
- moved U$1 4.14 mm to (24.8, 29.8), turned to 270 degrees
- moved C1 2.31 mm to (22.2, 29.8), turned to 90 degrees
- moved R2 0.95 mm to (31.1, 24.8), turned to 270 degrees
- moved C20 0.32 mm to (30.6, 27.1)
- moved C21 0.32 mm to (30.2, 29.2)
- moved U1 0.32 mm to (25.1, 22.9)
Connections:
- removed net AM_DRDY: U1.41
- removed net AM_INT1: U1.42
- removed net AM_INT2: U1.43
- removed net GPS_RESET: U1.14
- removed net GPS_RX: U1.13
- removed net GPS_STATUS: U1.11
- removed net GPS_TX: U1.12
- removed net GYRO_CS: U1.18
- removed net GYRO_INT1: U1.21
- removed net GYRO_INT2: U1.19
- removed net MISO: U1.16
- removed net MOSI: U1.17
- removed net SCK: U1.15
- removed net SCL: U1.45
- removed net SDA: U1.46
- removed net UART_RX: U1.31, X1.4
- removed net UART_TX: U1.30, X1.3
- new net +V: U$10.2, U$11.2, U$12.2, U$13.2, U$14.2, U$15.2, U$2.2, U$3.2, U$5.2, U$6.2, U$7.2, U$8.2, U$9.2
- new net N$10: RN2.7, U$8.3
- new net N$11: RN2.6, U$9.3
- new net N$12: RN2.5, U$10.3
- new net N$13: RN3.8, U$11.3
- new net N$14: RN3.7, U$12.3
- new net N$16: RN3.6, U$13.3
- new net N$17: RN3.5, U$14.3
- new net N$6: RN1.7, U$3.3
- new net N$7: RN1.6, U$5.3
- new net N$8: RN1.5, U$6.3
- new net N$9: RN2.8, U$7.3
- new net RC1: RN1.1, U1.29
- new net RC10: RN3.2, U1.12
- new net RC11: RN3.3, U1.10
- new net RC12: RN3.4, U1.11
- new net RC2: RN1.2, U1.31
- new net RC3: RN1.3, U1.42
- new net RC4: RN1.4, U1.45
- new net RC5: RN2.1, U1.19
- new net RC6: RN2.2, U1.18
- new net RC7: RN2.3, U1.17
- new net RC8: RN2.4, U1.16
- new net RC9: RN3.1, U1.13
- net +3V3: no longer R3.1
- net +5V: no longer X1.1
- net GND: now also U$10.1, U$11.1, U$12.1, U$13.1, U$14.1, U$15.1, U$2.1, U$3.1, U$5.1, U$6.1, U$7.1, U$8.1, U$9.1; no longer X1.2
- net N$3: now also RN1.8, U$2.3; no longer R3.2, U$1.1
Routing:
- net GND: track 0.00 -> 41.6 mm, vias 8 -> 10
- net UART_TX: track 41.2 -> 0.00 mm, vias 1 -> 0
- net UART_RX: track 36.8 -> 0.00 mm, vias 1 -> 0
- net +5V: track 51.4 -> 17.1 mm
- net +V: track 0.00 -> 31.7 mm
- net RC2: track 0.00 -> 26.2 mm, vias 0 -> 2
- net RC1: track 0.00 -> 25.9 mm, vias 0 -> 2
- net RC3: track 0.00 -> 25.6 mm, vias 0 -> 2
- net RC4: track 0.00 -> 24.4 mm, vias 0 -> 2
- net N$17: track 0.00 -> 14.2 mm, vias 0 -> 1
- net RC5: track 0.00 -> 12.7 mm
- net N$16: track 0.00 -> 12.6 mm, vias 0 -> 1
- net RC6: track 0.00 -> 11.5 mm
- net N$14: track 0.00 -> 10.9 mm
- net RC7: track 0.00 -> 10.5 mm
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