File: hw/RC_module.sch (EAGLE design)
At the start: 32 parts, among them U1 STM32F103CX, U5 LD3985XX, X1 MICROMATCH-4

Commit message: layout completed
Parts:
- removed R3: 100k, rcl:R-EU_R0603
- removed X1: MICROMATCH-4, tyco:MICROMATCH-4
- added RN1, RN2, RN3: (no value), dp_devices:RESISTOR_ARRAY_4
- added U$10, U$11, U$12, U$13, U$14, U$2, U$3, U$5, U$6, U$7, U$8, U$9: PINHD-3, connectors:PINHD-3
- added U$15: SCREWTERMINAL_3-3, connectors:SCREWTERMINAL_3-3
- C11: value 15pF -> 10n
Connections:
- removed net AM_DRDY: U1.PB5
- removed net AM_INT1: U1.PB6
- removed net AM_INT2: U1.PB7
- removed net GPS_RESET: U1.PA4
- removed net GPS_RX: U1.PA3
- removed net GPS_STATUS: U1.PA1
- removed net GPS_TX: U1.PA2
- removed net GYRO_CS: U1.PB0
- removed net GYRO_INT1: U1.PB10
- removed net GYRO_INT2: U1.PB1
- removed net MISO: U1.PA6
- removed net MOSI: U1.PA7
- removed net SCK: U1.PA5
- removed net SCL: U1.PB8
- removed net SDA: U1.PB9
- removed net UART_RX: U1.PA10, X1-4.S
- removed net UART_TX: U1.PA9, X1-3.S
- new net +V: U$10.P$2, U$11.P$2, U$12.P$2, U$13.P$2, U$14.P$2, U$15.P$2, U$2.P$2, U$3.P$2, U$5.P$2, U$6.P$2, U$7.P$2, U$8.P$2, U$9.P$2
- new net N$10: RN2B.2, U$8.P$3
- new net N$11: RN2C.2, U$9.P$3
- new net N$12: RN2D.2, U$10.P$3
- new net N$13: RN3A.2, U$11.P$3
- new net N$14: RN3B.2, U$12.P$3
- new net N$16: RN3C.2, U$13.P$3
- new net N$17: RN3D.2, U$14.P$3
- new net N$6: RN1B.2, U$3.P$3
- new net N$7: RN1C.2, U$5.P$3
- new net N$8: RN1D.2, U$6.P$3
- new net N$9: RN2A.2, U$7.P$3
- new net RC1: RN1A.1, U1.PA8
- new net RC10: RN3B.1, U1.PA2
- new net RC11: RN3C.1, U1.PA0/WKUP
- new net RC12: RN3D.1, U1.PA1
- new net RC2: RN1B.1, U1.PA10
- new net RC3: RN1C.1, U1.PB6
- new net RC4: RN1D.1, U1.PB8
- new net RC5: RN2A.1, U1.PB1
- new net RC6: RN2B.1, U1.PB0
- new net RC7: RN2C.1, U1.PA7
- new net RC8: RN2D.1, U1.PA6
- new net RC9: RN3A.1, U1.PA3
- net +3V3: no longer R3.1
- net +5V: no longer X1-1.S
- net GND: now also U$10.P$1, U$11.P$1, U$12.P$1, U$13.P$1, U$14.P$1, U$15.P$1, U$2.P$1, U$3.P$1, U$5.P$1, U$6.P$1, U$7.P$1, U$8.P$1, U$9.P$1; no longer X1-2.S
- net N$3: now also RN1A.2, U$2.P$3; no longer R3.2, U$1.TRI
